File: Assignment1/Assignment1.kicad_pcb (KiCad board)
At the start: 2 copper layers, 50 x 50 mm, 22 parts, among them J1 Conn_01x02_Pin, J2 Conn_01x02_Pin, U1 TPS51386RJNR, U2 LD39200PU33R

Commit message: First Assignment
Parts:
- moved J2 10.4 mm to (87.6, 72.6), turned to 180 degrees
- moved Cout1 6.71 mm to (79.7, 75.2)
- moved Cbyp1 6.69 mm to (84.7, 71.7)
- moved R_LDO_1 6.69 mm to (82.7, 71.8)
- moved U2 6.69 mm to (78.2, 71.6)
- moved R_LDO_2 5.93 mm to (82.8, 68.6), turned to -90 degrees
- moved Cin1 5.33 mm to (75.2, 70.9)
- moved R5 5.24 mm to (66.0, 75.2)
- moved C7 4.83 mm to (73.4, 70.9)
- moved C12 4.70 mm to (70.6, 75.2)
- moved L1 4.57 mm to (70.1, 71.6)
- moved C1 3.13 mm to (70.1, 67.8)
- moved R6 2.92 mm to (64.5, 77.0)
- moved R4 2.11 mm to (70.6, 77.0)
- moved R1 1.86 mm to (68.3, 67.8)
Routing:
- net /BuckStep_Vout: track 18.1 -> 11.8 mm
- net /Vout: track 14.7 -> 9.98 mm
- net /Buck_FB: track 12.3 -> 8.46 mm
- net Earth: track 3.99 -> 7.67 mm, vias 11 -> 12
- net /Buck_SW: track 7.45 -> 6.28 mm
- net Net-(U2-SENSE): track 8.23 -> 7.18 mm
- net Net-(C1-Pad1): track 2.80 -> 1.80 mm
- net /Buck_VBST: track 2.41 -> 3.27 mm
- net /Buck_Vin: track 11.4 -> 10.8 mm
- net Net-(C12-Pad1): track 2.41 -> 2.97 mm
