File: Assignment2/Assignment2.kicad_pcb (KiCad board)
At the start: 2 copper layers, 50 x 50 mm, 51 parts, among them J1 USB_B_Micro, J2 Conn_01x02, J3 Conn_01x03, J4 Conn_01x02, SW1 SW_Push, U1 RP2040, U2 NCP1117-3.3_SOT223, U3 W25Q128JVS, U4 ABM8-272-T3, U5 MAX98357A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

Commit message: footprint
Parts:
- added G***: LOGO, ba-gay.preety:ba-gay, F.Cu at (136.5, 84.5)
Other:
- board text added: "PCB Design Assignment 2 RP2040 & I²S"
