File: FinalProject/FinalProject.kicad_sch (KiCad schematic)
At the start: 51 parts, among them J1 USB_B_Micro, J2 Conn_01x02, J3 Conn_01x03, J4 Conn_01x02, SW1 SW_Push, U1 RP2040, U2 NCP1117-3.3_SOT223, U3 W25Q128JVS, U4 ABM8-272-T3, U5 MAX98357A, U6 VEML6040

Commit message: FinalProject Init
Other:
- added sheet USB Hub (untitled.kicad_sch)
Changed lines of the file:
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@@
+		)
+	)
+	(sheet
+		(at 85.09 168.91)
+		(size 210.82 111.76)
+		(exclude_from_sim no)
+		(in_bom yes)
+		(on_board yes)
+		(dnp no)
+		(fields_autoplaced yes)
+		(stroke
+			(width 0.1524)
+			(type solid)
+		)
+		(fill
+			(color 0 0 0 0.0000)
+		)
+		(property "Sheetname" "USB Hub"
+			(at 85.09 168.1984 0)
+			(effects
+				(font
+					(size 1.27 1.27)
+				)
+				(justify left bottom)
+			)
+		)
+		(property "Sheetfile" "untitled.kicad_sch"
+			(at 85.09 281.2546 0)
+			(effects
+				(font
+					(size 1.27 1.27)
+				)
+				(justify left top)
+			)
+		)
+		(instances
+			(project "FinalProject"
+				(path "/ec64d11f-31de-42eb-b4e8-dd7a6ad77b85"
+					(page "2")
+				)
+			)
 		)
 	)

Commit message: Final Project Schematic
Parts:
- removed C1, C17, C2: 10μF, Capacitor_SMD:C_0603_1608Metric, symbol Device:C
- removed C10, C11, C12, C13, C14, C15, C16, C21, C7, C8: 100nF, Capacitor_SMD:C_0603_1608Metric, symbol Device:C
- removed C18, C19: 0.1μF, Capacitor_SMD:C_0603_1608Metric, symbol Device:C
- removed C20: 200pF, Capacitor_SMD:C_0603_1608Metric, symbol Device:C
- removed C3: 100μF, Capacitor_SMD:C_0603_1608Metric, symbol Device:C
- removed C4, C5: 15pF, Capacitor_SMD:C_0402_1005Metric, symbol Device:C
- removed C6, C9: 1μF, Capacitor_SMD:C_0402_1005Metric, symbol Device:C
- removed D1, D2: LED, LED_SMD:LED_0603_1608Metric, symbol Device:LED
- removed H1, H2, H3, H4: MountingHole, MountingHole:MountingHole_2.7mm_M2.5, symbol Mechanical:MountingHole
- removed J1: USB_B_Micro, Connector_USB:USB_Micro-B_Amphenol_10103594-0001LF_Horizontal, symbol Connector:USB_B_Micro
- removed J2, J4: Conn_01x02, Connector_PinSocket_2.54mm:PinSocket_1x02_P2.54mm_Vertical, symbol Connector_Generic:Conn_01x02
- removed J3: Conn_01x03, Connector_PinSocket_2.54mm:PinSocket_1x03_P2.54mm_Vertical, symbol Connector_Generic:Conn_01x03
- removed MK1: SPH0645LM4H, Sensor_Audio:Knowles_SPH0645LM4H-6_3.5x2.65mm, symbol Sensor_Audio:SPH0645LM4H
- removed R1: 1kΩ, Resistor_SMD:R_0603_1608Metric, symbol Device:R
- removed R10, R9: 2.2kΩ, Resistor_SMD:R_0603_1608Metric, symbol Device:R
- removed R11, R12: 150Ω, Resistor_SMD:R_0603_1608Metric, symbol Device:R
- removed R2: DNF, Resistor_SMD:R_0603_1608Metric, symbol Device:R
- removed R3, R4: 27Ω, Resistor_SMD:R_0603_1608Metric, symbol Device:R
- removed R5: 1MΩ, Resistor_SMD:R_0603_1608Metric, symbol Device:R
- removed R6, R7, R8: 51Ω, Resistor_SMD:R_0603_1608Metric, symbol Device:R
- removed SW1: SW_Push, Button_Switch_THT:SW_PUSH_1P1T_6x3.5mm_H4.3_APEM_MJTP1243, symbol Switch:SW_Push
- removed U1: RP2040, Package_DFN_QFN:QFN-56-1EP_7x7mm_P0.4mm_EP3.2x3.2mm, symbol MCU_RaspberryPi:RP2040
- removed U2: NCP1117-3.3_SOT223, Package_TO_SOT_SMD:SOT-223-3_TabPin2, symbol Regulator_Linear:NCP1117-3.3_SOT223
- removed U3: W25Q128JVS, Package_SO:SOIC-8_5.3x5.3mm_P1.27mm, symbol Memory_Flash:W25Q128JVS
- removed U4: ABM8-272-T3, ABM8-272-T3:ABM8-272-T3, symbol ABM8-272-T3:ABM8-272-T3
- removed U5: MAX98357A, Package_DFN_QFN:TQFN-16-1EP_3x3mm_P0.5mm_EP1.23x1.23mm, symbol Audio:MAX98357A
- removed U6: VEML6040, VEML6040:VISHAY_VEML6040_1.25X2X1, symbol VEML6040:VEML6040
- added C36, C37, C38, C39, C40, C85, C86, C87, C88, C89, C90: 100nF, Capacitor_SMD:C_0603_1608Metric, symbol Device:C
- added C41, C42: 10μF, Capacitor_SMD:C_0603_1608Metric, symbol Device:C
- added C43, C44: 10uF, Capacitor_SMD:C_0603_1608Metric, symbol Device:C
- added C5, C6: 100uF, Capacitor_SMD:C_0603_1608Metric, symbol Device:C_US
- added C69, C70: 27pF, Capacitor_SMD:C_0603_1608Metric, symbol Device:C
- added C71: 22nF, Capacitor_SMD:C_0603_1608Metric, symbol Device:C
- added C75, C79, C80, C81, C82, C83, C84, C92, C93, C94, C95, C96, C97, C98, C99: 0.1uF, Capacitor_SMD:C_0603_1608Metric, symbol Device:C
- added C76, C91: 10nF, Capacitor_SMD:C_0603_1608Metric, symbol Device:C
- added D1: SMBJ33CA, DIONM5436X261N, symbol SMBJ33CA:SMBJ33CA
- added J12, J13: USB3_A, symbol Connector:USB3_A
- added J14: USB_C_Receptacle, symbol Connector:USB_C_Receptacle
- added J5: ARJM11D7-502-AB-EW2, ARJM11D7-502-AB-EW2:ABRACON_ARJM11D7-502-AB-EW2, symbol ARJM11D7-502-AB-EW2:ARJM11D7-502-AB-EW2
- added J6: DCJ200-10-A-XX-K_REVA, DCJ200-10-A-XX-K_REVA:GCT_DCJ200-10-A-XX-K_REVA, symbol DCJ200-10-A-XX-K_REVA:DCJ200-10-A-XX-K_REVA
- added L1: 2.2uH, symbol Device:L
- added Q1: NTTFS5C673NLTAG, NVTFS6H854NTAG, symbol NTTFS5C673NLTAG:NTTFS5C673NLTAG
- added R13: 100k, Resistor_SMD:R_0603_1608Metric, symbol Device:R
- added R14: 75k, Resistor_SMD:R_0603_1608Metric, symbol Device:R
- added R15: 200k, Resistor_SMD:R_0603_1608Metric, symbol Device:R
- added R19: 200K, Resistor_SMD:R_0603_1608Metric, symbol Device:R
- added R20: 4.7k, Resistor_SMD:R_0603_1608Metric, symbol Device:R
- added R21: 900K, Resistor_SMD:R_0603_1608Metric, symbol Device:R
- added R39: 2.49K, Resistor_SMD:R_0603_1608Metric, symbol Device:R
- added R40: 470R, Resistor_SMD:R_0603_1608Metric, symbol Device:R
- added R41: 0R, Resistor_SMD:R_0603_1608Metric, symbol Device:R
- added U1: RTL8153B-VB-CG, RTL8153B-VB-CG:QFN40P500X500X90-41N, symbol RTL8153B-VB-CG:RTL8153B-VB-CG
- added U13: HD3SS3220IRNHR, RNH0030A, symbol 2025-04-19_06-45-11:HD3SS3220IRNHR
- added U14: NCP1117-3.3_SOT223, Package_TO_SOT_SMD:SOT-223-3_TabPin2, symbol Regulator_Linear:NCP1117-3.3_SOT223
- added U3: LM74700, Package_TO_SOT_SMD:SOT-23-6, symbol Power_Management:LM74700
- added U7: TPS62160DGKR, DGK0008A_N, symbol 2025-04-23_17-50-30:TPS62160DGKR
- added Y2: ABLS-25.000MHZ-B2F-T, ABLS-25.000MHZ-B2F-T:XTAL_ABLS-25.000MHZ-B2F-T, symbol ABLS-25.000MHZ-B2F-T:ABLS-25.000MHZ-B2F-T
Connections:
- net +1V1: now also C44.1, C79.2, C80.2, C81.2, C82.2, C83.2, C84.2, C92.2, L1.2, R13.2, R14.2, U1.14 (U3VDD10), U1.19 (U2VDD10), U1.22 (DVDD10_UPS), U1.3 (AVDD10), U1.34 (DVDD10), U1.37 (AVDD10__2), U1.8 (AVDD10__1), U7.6 (VOS)
- net +3.3V: now also C42.1, C93.2, C94.2, C95.2, C96.2, C97.2, C98.2, R19.1, R40.1, U1.11 (AVDD33), U1.20 (AVDD33__1), U1.23 (DVDD33), U1.33 (DVDD33__1), U1.39 (AVDD33__2), U1.40 (AVDD33__3), U13.8 (VCC33), U14.2 (VO)
- net +5V: now also C36.2, C41.1, C43.1, C5.1, C6.1, C75.2, C76.2, Q1.5 (D_1), Q1.6 (D_2), Q1.7 (D_3), Q1.8 (D_4), U1.21 (VDD5), U13.30 (VDD5), U14.3 (VI), U3.4 (CATHODE), U7.2 (VIN), U7.3 (EN)
- net GND: now also C36.1, C41.2, C42.2, C43.2, C44.2, C5.2, C6.2, C69.2, C70.1, C70.2, C71.2, C75.1, C76.1, C79.1, C80.1, C81.1, C82.1, C83.1, C84.1, C91.2, C92.1, C93.1, C94.1, C95.1, C96.1, C97.1, C98.1, D1.1, J12.10 (SHIELD), J12.4 (GND), J12.7 (DRAIN), J13.10 (SHIELD), J13.4 (GND), J13.7 (DRAIN), J14.A1 (GND), J14.A12 (GND), J14.B1 (GND), J14.B12 (GND), J14.S1 (SHIELD), J6.2, J6.3, R15.2, R20.1, R39.2, R41.1, U1.25 (EEDI/SPIDI/ENSWREG), U1.29 (GND), U1.36 (CKXTAL2), U1.41 (GND__1), U13.12 (EN_MUX_N), U13.13 (GND), U13.28 (GND), U13.29 (EN_CC_N), U13.31 (PAD), U14.1 (GND), U3.2 (GND), U7.1 (PGND), U7.4 (AGND), Y2.2
- new net: Q1.4 (G), U3.5 (GATE)
- new net: C87.1, J13.8 (SSTX-)
- new net: C88.1, J13.9 (SSTX+)
- new net: C90.1, U1.12 (U3SSTXN)
- new net: R21.2, U13.5 (VBUS_DET)
- new net: J5.P11, J5.P13, R40.2
- new net: C91.1, J5.S1 (SHIELD), J5.S2 (SHIELD), R41.2
- new net: C85.1, J12.8 (SSTX-)
- new net: C39.1, U13.21 (TX2P)
- new net: C86.1, J12.9 (SSTX+)
- new net: C38.1, U13.16 (TX1N)
- new net: C69.1, U1.35 (CKXTAL1), Y2.1
- new net: C89.1, U1.13 (U3SSTXP)
- new net: R39.1, U1.38 (RSET)
- new net: C40.1, U13.20 (TX2N)
- new net: R20.2, U13.4 (PORT)
- new net: R13.1, U7.8 (PG)
- new net: R19.2, U13.11 (DIR)
- new net: R14.1, R15.1, U7.5 (FB)
- new net: L1.1, U7.7 (SW)
- new net: C37.1, U13.17 (TX1P)
- new net: C99.2, U3.1 (VCAP)
- new net DN1_D+: U1.18 (U2DP)
- new net DN1_D-: U1.17 (U2DM)
- new net DN1_RXN: U1.15 (U3SSRXN)
- new net DN1_RXP: U1.16 (U3SSRXP)
- new net DN1_TXN: C89.2
- new net DN1_TXP: C90.2
- new net DN2_D+: J13.3 (D+)
- new net DN2_D-: J13.2 (D-)
- new net DN2_RXN: J13.5 (SSRX-)
- new net DN2_RXP: J13.6 (SSRX+)
- new net DN2_TXN: C87.2
- new net DN2_TXP: C88.2
- new net DN2_VBUS: J13.1 (VBUS)
- new net DN3_D+: J12.3 (D+)
- new net DN3_D-: J12.2 (D-)
- new net DN3_RXN: J12.5 (SSRX-)
- new net DN3_RXP: J12.6 (SSRX+)
- new net DN3_TXN: C85.2
- new net DN3_TXP: C86.2
- new net DN3_VBUS: J12.1 (VBUS)
- new net ETH_LED0: J5.P14, U1.32 (LED0/SPICSB)
- new net ETH_LED1: U1.30 (EESK/LED1/SPISCK)
- new net ETH_LED2: J5.P12, U1.24 (EEDO/LED2/SPISDO/LANWAKEB/GPIO)
- new net IN_CC1: J14.A5 (CC1), U13.2 (CC1)
- new net IN_CC2: J14.B5 (CC2), U13.1 (CC2)
- new net IN_RX1+: J14.B11 (RX1+), U13.15 (RX1P)
- new net IN_RX1-: J14.B10 (RX1-), U13.14 (RX1N)
- new net IN_RX2+: J14.A11 (RX2+), U13.19 (RX2P)
- new net IN_RX2-: J14.A10 (RX2-), U13.18 (RX2N)
- new net IN_TX1+: C37.2, J14.A2 (TX1+)
- new net IN_TX1-: C38.2, J14.A3 (TX1-)
- new net IN_TX2+: C39.2, J14.B2 (TX2+)
- new net IN_TX2-: C40.2, J14.B3 (TX2-)
- new net Power_Supply_5.0: C71.1, C99.1, D1.2, J6.1, Q1.1 (S_1), Q1.2 (S_2), Q1.3 (S_3), U3.3 (EN), U3.6 (ANODE)
- new net TD1+: J5.P1 (TD1+), U1.1 (MDIP0)
- new net TD1-: J5.P2 (TD1-), U1.2 (MDIN0)
- new net TD2+: J5.P3 (TD2+), U1.4 (MDIP1)
- new net TD2-: J5.P4 (TD2-), U1.5 (MDIN1)
- new net TD3+: J5.P7 (TD3+), U1.6 (MDIP2)
- new net TD3-: J5.P8 (TD3-), U1.7 (MDIN2)
- new net TD4+: J5.P9 (TD4+), U1.9 (MDIP3)
- new net TD4-: J5.P10 (TD4-), U1.10 (MDIN3)
- new net UP_D+: J14.A6 (D+), J14.B6 (D+)
- new net UP_D-: J14.A7 (D-), J14.B7 (D-)
- new net UP_RXN: U13.10 (RXN)
- new net UP_RXP: U13.9 (RXP)
- new net UP_TXN: U13.7 (TXN)
- new net UP_TXP: U13.6 (TXP)
- new net UP_VBUS: J14.A4 (VBUS), J14.A9 (VBUS), J14.B4 (VBUS), J14.B9 (VBUS), R21.1
- no-connect marks 21 -> 19
Other:
- removed sheet USB Hub
- added sheet RP2040 (RP2040.kicad_sch)
- added sheet USB HUB (USB_HUB.kicad_sch)
- note added: "5.0V to 1.1V"
- note added: "5.0V to 3.3V"
- note added: "DownStream USB-C Interface (CH2)"
- note added: "Downstream USB"
- note added: "Peripheral"
- note added: "Power Input"
- note added: "Power Management Unit"
- note added: "RJ-45 Ethernet Interface"
- note added: "Upstream USB-C Interface"
- note removed: "C6 must be close to VREG_VOUT"
- note removed: "C9 must be close to VREG_VIN"
- note removed: "Color Sensor Module"
- note removed: "Crystal Unit"
- note removed: "Decoupling (C19) and RF Filter (C20) capacitor should be close to the microphone (RF Filter be closest) and use short, wide trace to minimize inductance."
- note removed: "Flash Memory Unit"
- note removed: "LED Module"
- note removed: "Microphone Unit"
- note removed: "Power and Data Unit"
- note removed: "RP2040 Unit"
- note removed: "Reset Unit"
- note removed: "Todo List 1. Add Input Audio Unit - DONE 2. Add Color Sensor Unit - DONE 3. Fill in the Footprint - DONE (Probably) 4. Route and place"
- note removed: "Use VIA to connect microphone's ground pad to other layer's ground pane."

Commit message: fix schematic
Parts:
- removed C43, C44: 10uF, Capacitor_SMD:C_0603_1608Metric, symbol Device:C
- removed C86, C87, C88: 100nF, Capacitor_SMD:C_0603_1608Metric, symbol Device:C
- removed C91: 10nF, Capacitor_SMD:C_0603_1608Metric, symbol Device:C
- removed J12, J13: USB3_A, symbol Connector:USB3_A
- removed J14: USB_C_Receptacle, symbol Connector:USB_C_Receptacle
- removed L1: 2.2uH, symbol Device:L
- removed R13: 100k, Resistor_SMD:R_0603_1608Metric, symbol Device:R
- removed R14: 75k, Resistor_SMD:R_0603_1608Metric, symbol Device:R
- removed R15: 200k, Resistor_SMD:R_0603_1608Metric, symbol Device:R
- removed R41: 0R, Resistor_SMD:R_0603_1608Metric, symbol Device:R
- removed U7: TPS62160DGKR, DGK0008A_N, symbol 2025-04-23_17-50-30:TPS62160DGKR
- added C100: 22uF, Capacitor_SMD:C_0603_1608Metric, symbol Device:C
- added C101: 10uF, Capacitor_SMD:C_0603_1608Metric, symbol Device:C
- added C102, C103, C104, C105: 100nF, Capacitor_SMD:C_0603_1608Metric, symbol Device:C
- added C106: 0.1uF, Capacitor_SMD:C_0603_1608Metric, symbol Device:C
- added C7: 100uF, Capacitor_SMD:C_0603_1608Metric, symbol Device:C_US
- added D2: SMBJ33CA, DIONM5436X261N, symbol SMBJ33CA:SMBJ33CA
- added J1: 10152803-00011LF, 10152803-00011LF:AMPHENOL_10152803-00011LF, symbol 10152803-00011LF:10152803-00011LF
- added J2, J3: GSB4111312HR, GSB4111312HR:AMPHENOL_GSB4111312HR, symbol GSB4111312HR:GSB4111312HR
- added L2: 1uH, Inductor_SMD:L_1008_2520Metric, symbol Device:L
- added Q2: NTTFS5C673NLTAG, NVTFS6H854NTAG, symbol NTTFS5C673NLTAG:NTTFS5C673NLTAG
- added R45: 11K, Resistor_SMD:R_0603_1608Metric, symbol Device:R
- added R46: 26.1K, Resistor_SMD:R_0603_1608Metric, symbol Device:R
- added U4: TPS62902RPJR, QFN_902RPJR_TEX, symbol 2025-04-27_02-17-23:TPS62902RPJR
- added U5: LM74700, Package_TO_SOT_SMD:SOT-23-6, symbol Power_Management:LM74700
- C85: value 100nF -> 22nF
Connections:
- net +1V1: now also C100.1, L2.2, U4.3 (VOS)
- net +5V: now also C101.2, U4.5 (EN), U4.6 (VIN)
- net DN2_D+: now also J2.3 (D+)
- net DN2_D-: now also J2.2 (D-)
- net DN2_RXN: now also J2.5 (SSRX-)
- net DN2_RXP: now also J2.6 (SSRX+)
- net DN2_TXN: now also C102.2
- net DN2_TXP: now also C103.2
- net DN2_VBUS: now also J2.1 (VBUS)
- net DN3_D+: now also J3.3 (D+)
- net DN3_D-: now also J3.2 (D-)
- net DN3_RXN: now also J3.5 (SSRX-)
- net DN3_RXP: now also J3.6 (SSRX+)
- net DN3_TXN: now also C104.2; no longer C85.2
- net DN3_TXP: now also C105.2
- net DN3_VBUS: now also J3.1 (VBUS)
- net GND: now also C85.2, J5.S1 (SHIELD), J5.S2 (SHIELD), C100.2, C101.1, C7.2, D2.1, J1.A1 (GND_A), J1.A12 (GND_A__1), J1.B1 (GND_B), J1.B12 (GND_B__1), J1.S1 (SHIELD), J1.S2 (SHIELD__1), J1.S3 (SHIELD__2), J1.S4 (SHIELD__3), J2.4 (GND), J2.7 (GND_DRAIN), J2.SH1 (SHIELD), J2.SH2 (SHIELD__1), J3.4 (GND), J3.7 (GND_DRAIN), J3.SH1 (SHIELD), J3.SH2 (SHIELD__1), R45.1, R46.1, U4.4 (GND), U5.2 (GND)
- net IN_CC1: now also J1.A5 (CC1)
- net IN_CC2: now also J1.B5 (CC2)
- net IN_RX1+: now also J1.B11 (SSRXP1)
- net IN_RX1-: now also J1.B10 (SSRXN1)
- net IN_RX2+: now also J1.A11 (SSRXP2)
- net IN_RX2-: now also J1.A10 (SSRXN2)
- net IN_TX1+: now also J1.A2 (SSTXP1)
- net IN_TX1-: now also J1.A3 (SSTXN1)
- net IN_TX2+: now also J1.B2 (SSTXP2)
- net IN_TX2-: now also J1.B3 (SSTXN2)
- net UP_D+: now also J1.A6 (DP1), J1.B6 (DP2)
- net UP_D-: now also J1.A7 (DN1), J1.B7 (DN2)
- net UP_VBUS: now also C85.1, C106.1, D2.2, J1.A4 (VBUS_A), J1.A9 (VBUS_A__1), J1.B4 (VBUS_B), J1.B9 (VBUS_B__1), Q2.1 (S_1), Q2.2 (S_2), Q2.3 (S_3), U5.3 (EN), U5.6 (ANODE); no longer R21.1
- new net: C106.2, U5.1 (VCAP)
- new net: Q2.4 (G), U5.5 (GATE)
- new net: L2.1, U4.2 (SW)
- new net: C103.1, J2.9 (SSTX+)
- new net: C102.1, J2.8 (SSTX-)
- new net: C104.1, J3.8 (SSTX-)
- new net: R45.2, U4.9 (FB/VSET)
- new net: C105.1, J3.9 (SSTX+)
- new net: R46.2, U4.7 (MODE/S-CONF)
- new net UP_VBUS_DIODE: C7.1, Q2.5 (D_1), Q2.6 (D_2), Q2.7 (D_3), Q2.8 (D_4), R21.1, U5.4 (CATHODE)
- no-connect marks 19 -> 21

Commit message: fix smt
Parts:
- J1: footprint 10152803-00011LF:AMPHENOL_10152803-00011LF -> 10152803_00011LF:AMPHENOL_10152803-00011LF
- Y2: footprint ABLS-25.000MHZ-B2F-T:XTAL_ABLS-25.000MHZ-B2F-T -> ABLS_25_000MHZ_B2F_T:XTAL_ABLS-25.000MHZ-B2F-T
Changed lines of the file:
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@@
 			)
 		)
-		(property "Footprint" "ABLS-25.000MHZ-B2F-T:XTAL_ABLS-25.000MHZ-B2F-T"
+		(property "Footprint" "ABLS_25_000MHZ_B2F_T:XTAL_ABLS-25.000MHZ-B2F-T"
 			(at 256.54 229.87 0)
 			(effects
@@
 			)
 		)
-		(property "Footprint" "10152803-00011LF:AMPHENOL_10152803-00011LF"
+		(property "Footprint" "10152803_00011LF:AMPHENOL_10152803-00011LF"
 			(at 49.53 52.07 0)
 			(effects

Commit message: route pi part 1
Parts:
- added H1, H2, H3, H4: MountingHole, MountingHole:MountingHole_2.7mm_M2.5, symbol Mechanical:MountingHole
Connections:
- net GND: no longer C70.1, U1.36 (CKXTAL2), Y2.2
- new net: C70.1, U1.36 (CKXTAL2), Y2.2
Other:
- note added: "Ethernet Module"
- note added: "Power Switching"
- note added: "Submodules"
- moved on the sheet: C102, C103, C104, C105, C106, C5, C6, C69, C7, C70, C71, C75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
