File: FinalProject/FinalProject.kicad_sch (KiCad schematic)
At the start: 58 parts, among them J1 GSB4111312HR, J2 GSB4111312HR, J3 GSB4111312HR, J5 ARJM11D7-502-AB-EW2, J6 DCJ200-10-A-XX-K_REVA, Q1 NTTFS5C673NLTAG, Q2 NTTFS5C673NLTAG, U1 RTL8153B-VB-CG, U14 NCP1117-3.3_SOT223, U3 LM74700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

Commit message: update big capacitors footprint to use bigger than 0603
Parts:
- C5, C6, C7: footprint Capacitor_SMD:C_0603_1608Metric -> Capacitor_SMD:C_1206_3216Metric
Changed lines of the file:
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@@
 			)
 		)
-		(property "Footprint" "Capacitor_SMD:C_0603_1608Metric"
+		(property "Footprint" "Capacitor_SMD:C_1206_3216Metric"
 			(at 369.57 226.06 0)
 			(effects
@@
 			)
 		)
-		(property "Footprint" "Capacitor_SMD:C_0603_1608Metric"
+		(property "Footprint" "Capacitor_SMD:C_1206_3216Metric"
 			(at 440.69 331.47 0)
 			(effects
@@
 			)
 		)
-		(property "Footprint" "Capacitor_SMD:C_0603_1608Metric"
+		(property "Footprint" "Capacitor_SMD:C_1206_3216Metric"
 			(at 308.61 331.47 0)
 			(effects
