File: FinalProject/RP2040.kicad_sch (KiCad schematic)
At the start: 50 parts, among them J10 Conn_01x02, J7 Conn_01x02, J9 Conn_01x03, SW2 SW_Push, U10 NCP1117-3.3_SOT223, U11 RP2040, U15 VEML6040, U16 MAX98357A, U8 ABM8-272-T3, U9 W25Q128JVS

Commit message: fix schematic
Parts:
- removed C48, C49: 10μF, Capacitor_SMD:C_0603_1608Metric, symbol Device:C
- removed U10: NCP1117-3.3_SOT223, Package_TO_SOT_SMD:SOT-223-3_TabPin2, symbol Regulator_Linear:NCP1117-3.3_SOT223

Commit message: route pi part 1
Parts:
- removed H5, H6, H7, H8: MountingHole, MountingHole:MountingHole_2.7mm_M2.5, symbol Mechanical:MountingHole
Connections:
- net GPIO0: now also U11.35 (GPIO23); no longer U11.2 (GPIO0)
- net GPIO1: now also U11.36 (GPIO24); no longer U11.3 (GPIO1)
- net GPIO2: now also U11.37 (GPIO25); no longer U11.4 (GPIO2)
- net GPIO3: now also U11.32 (GPIO21); no longer U11.5 (GPIO3)
- net GPIO4: now also U11.34 (GPIO22); no longer U11.6 (GPIO4)
- net GPIO5: now also U11.31 (GPIO20); no longer U11.7 (GPIO5)
- net GPIO6: now also U11.30 (GPIO19); no longer U11.8 (GPIO6)
- net GPIO7: now also U11.29 (GPIO18); no longer U11.9 (GPIO7)
- net USB_DP: now reaches R25.2, U11.47 (USB_DP)
- net USB_DN: now reaches R26.2, U11.46 (USB_DM)
Other:
- note removed: "Todo List 1. Add Input Audio Unit - DONE 2. Add Color Sensor Unit - DONE 3. Fill in the Footprint - DONE (Probably) 4. Route and place"
- moved on the sheet: J9

Commit message: update big capacitors footprint to use bigger than 0603
Parts:
- C50: footprint Capacitor_SMD:C_0603_1608Metric -> Capacitor_SMD:C_1206_3216Metric
Changed lines of the file:
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@@
 			)
 		)
-		(property "Footprint" "Capacitor_SMD:C_0603_1608Metric"
+		(property "Footprint" "Capacitor_SMD:C_1206_3216Metric"
 			(at 77.1652 77.47 0)
 			(effects
